File: PCB/DoseManager/DoseManager.brd (EAGLE design)
At the start: 100.1 x 41.7 mm, 45 parts, among them J1 POWER_JACKPTH_LOCK, J3 RJ11, J4 RJ11, J5 RJ11, J6 RJ11, Q1 S8050, T2 S8050, X3 miniUSB, Y1 12MHz

Commit message: added panel and start of Lighting controller
Parts:
- removed C16: 10uF, SparkFun-Capacitors:0805
- removed C3: 10uF, microbuilder:0805-NO
- removed C6: 1uF, microbuilder:0805-NO
- removed Q1, T2: S8050, transistor:SOT23-BEC
- removed R1, R4: 470, LowPowerLab:0805
- removed R8, R9: 10k, LowPowerLab:0805
- removed U$4: CH340G, ch340g:SOIC16
- removed X3: miniUSB, microbuilder:USB-MINIB_LARGER
- removed Y1: 12MHz, SparkFun:RESONATOR-SMD
- added D2, D4: B120B-13-F, SparkFun-DiscreteSemi:SMB-DIODE
- added FLASH: (no value), SparkFun-Electromechanical:TACTILE_SWITCH_SMD
- added U$2: LOGO_GROBOTICS-S, 1_Skips:GROBOTICS-S
- added X5: (no value), con-conrad:733980-62
- J1: value POWER_JACKPTH_LOCK -> RJ45; device SparkFun-Connectors:POWER_JACK_PTH_LOCK -> SparkFun-Connectors:RJ45-8
- moved U$20 81.2 mm to (8.10, 0.64)
- moved C36 25.2 mm to (27.3, 28.1)
- moved L2 20.9 mm to (24.9, 31.9), turned to 0 degrees
- moved R43 20.6 mm to (23.0, 27.9)
- moved F1 20.6 mm to (15.2, 26.2)
- moved J1 20.1 mm to (6.35, 15.2), turned to 270 degrees
- moved R7 19.7 mm to (8.89, 38.1)
- moved R13 17.1 mm to (13.3, 34.1), turned to 180 degrees
- moved C9 17.1 mm to (19.1, 36.8)
- moved D1 17.1 mm to (15.2, 24.1), turned to 180 degrees
- moved R6 16.9 mm to (24.1, 38.1), turned to 270 degrees
- moved R3 15.2 mm to (15.2, 29.2)
- moved R5 14.0 mm to (21.6, 38.1)
- moved C10 14.0 mm to (7.62, 26.7)
- moved C12 14.0 mm to (7.62, 31.8)
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Connections:
- removed net +3V3: C3.1, C6.1, U$4.16, U$4.4
- removed net 12_TEMP: U1.GPIO12
- removed net 14_SCK: U1.GPIO14
- removed net 15: R3.2, U1.GPIO15
- removed net 3.3V: C12.1, OKI.OUT
- removed net A-STEP: U$6.STEP
- removed net B-STEP: U$1.STEP
- removed net C-STEP: U$5.STEP
- removed net D-STEP: U$7.STEP
- removed net DIR: U$1.DIR, U$5.DIR, U$6.DIR, U$7.DIR
- removed net ESP_DSLEEP: U1.GPIO16
- removed net FLOATS: J3.4, J4.4, J5.4, J6.4
- removed net GND: C1.-, C10.2, C12.2, C3.2, C4.-, C5.-, C6.2, C7.-, J1.GND, J3.6, J4.6, J5.6, J6.6, OKI.GND, U$1.GND, U$1.GND@0, U$4.1, U$5.GND, U$5.GND@0, U$6.GND, U$6.GND@0, U$7.GND, U$7.GND@0, X3.GND, X3.GND1, X3.GND2, X3.GND3, X3.GND4, Y1.2
- removed net N$13: R1.2, U$4.2
- removed net N$2: U$4.8, Y1.3
- removed net N$29: Q1.B, R8.1
- removed net N$30: R9.1, T2.B
- removed net N$31: Q1.E, R9.2, U$4.13
- removed net N$4: U$4.5, X3.D+
- removed net N$5: R8.2, T2.E, U$4.14
- removed net N$6: U$4.7, Y1.1
- removed net N$7: R4.2, U$4.3
- removed net PROBE_SCL: U1.GPIO5
- removed net PROBE_SDA: U1.GPIO4
- removed net VBUS1: D1.2, X3.VBUS
- new net 12_FLOATS: J3.4, J4.4, J5.4, J6.4, U1.GPIO12
- new net 14_A-STEP: U$6.STEP, U1.GPIO14
- new net 15_DIR: R3.2, U$1.DIR, U$5.DIR, U$6.DIR, U$7.DIR, U1.GPIO15
- new net 16_B-STEP: U$1.STEP, U1.GPIO16
- new net 4_C-STEP: U$5.STEP, U1.GPIO4
- new net 5V: D1.2, J1.1
- new net 5_D-STEP: U$7.STEP, U1.GPIO5
- net +12V: now also D2.C
- net ESP_3.3V: now also C12.1, OKI.OUT, U$1.VDD, U$5.VDD, U$6.VDD, U$7.VDD
- net ESP_FLASH: now also FLASH.1, J1.2; no longer Q1.C
- net ESP_GND: now also C1.-, C10.2, C12.2, C4.-, C5.-, C7.-, FLASH.4, J1.6, J1.7, J3.6, J4.6, J5.6, J6.6, OKI.GND, U$1.GND, U$1.GND@0, U$5.GND, U$5.GND@0, U$6.GND, U$6.GND@0, U$7.GND, U$7.GND@0, X5.2
- net ESP_RST: now also J1.3; no longer T2.C
- net ESP_RX: now also J1.4; no longer R4.1
- net ESP_TX: now also J1.5; no longer R1.1
- net N$3: now also D2.A, D4.A, X5.1; no longer U$4.6, X3.D-
- net VCC: now also D4.C; no longer J1.PWR, U$1.VDD, U$5.VDD, U$6.VDD, U$7.VDD
Routing:
- net ESP_3.3V: track 0.00 -> 181.1 mm, vias 0 -> 2
- net +12V: track 0.00 -> 96.4 mm
- net 2_ENABLE: track 0.00 -> 94.8 mm, vias 0 -> 2
- net 5_D-STEP: track 0.00 -> 93.3 mm, vias 0 -> 2
- net 12_FLOATS: track 0.00 -> 81.9 mm, vias 0 -> 1
- net 4_C-STEP: track 0.00 -> 78.1 mm, vias 0 -> 3
- net 15_DIR: track 0.00 -> 77.0 mm, vias 0 -> 2
- net ESP_RST: track 0.00 -> 59.3 mm, vias 0 -> 2
- net ESP_FLASH: track 0.00 -> 30.4 mm, vias 0 -> 1
- net ESP_TX: track 0.00 -> 29.9 mm
- net ESP_RX: track 0.00 -> 29.7 mm
- net 16_B-STEP: track 0.00 -> 27.5 mm
- net N$26: track 0.00 -> 20.7 mm
- net N$44: track 0.00 -> 20.7 mm
- net N$40: track 0.00 -> 20.7 mm
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- added copper zone on layer 1, net ESP_GND
- added copper zone on layer 16, net ESP_GND
Other:
- board size 100.1 x 41.7 mm -> 100.3 x 41.9 mm
- board text added: "6/25/17"
- board text added: "Dose Control v1 GroBotics.io"
