File: PCB/DoseManager/DoseManager.sch (EAGLE design)
At the start: 44 parts, among them J1 POWER_JACKPTH_LOCK, J3 RJ11, J4 RJ11, J5 RJ11, J6 RJ11, Q1 S8050, T2 S8050, X3 miniUSB, Y1 12MHz

Commit message: added panel and start of Lighting controller
Parts:
- removed C16: 10uF, SparkFun-Capacitors:CAP0805
- removed C3: 10uF, microbuilder:CAP_CERAMIC0805-NOOUTLINE
- removed C6: 1uF, microbuilder:CAP_CERAMIC0805-NOOUTLINE
- removed Q1, T2: S8050, transistor:BC817-16LT1-NPN-SOT23-BEC
- removed R1, R4: 470, LowPowerLab:RESISTOR0805
- removed R8, R9: 10k, LowPowerLab:RESISTOR0805
- removed U$4: CH340G, ch340g:CH340G
- removed X3: miniUSB, microbuilder:USBMINIBLARGE
- removed Y1: 12MHz, SparkFun:RESONATORSMD
- added D2, D4: B120B-13-F, SparkFun-DiscreteSemi:DIODESMB
- added FLASH: (no value), SparkFun-Electromechanical:TAC_SWITCHSMD
- added U$2: LOGO_GROBOTICS-S, 1_Skips:LOGO_GROBOTICS-S
- added X5: (no value), con-conrad:733980-62
- J1: value POWER_JACKPTH_LOCK -> RJ45; device SparkFun-Connectors:POWER_JACKPTH_LOCK -> SparkFun-Connectors:RJ45-8
Connections:
- removed net +3V3: C3.1, C6.1, U$4.V3, U$4.VCC
- removed net 12_TEMP: U1.12-MISO
- removed net 14_SCK: U1.14-SCK
- removed net 15: R3.2, U1.SS-15
- removed net 3.3V: C12.1, OKI.OUT
- removed net A-STEP: U$6.STEP
- removed net B-STEP: U$1.STEP
- removed net C-STEP: U$5.STEP
- removed net D-STEP: U$7.STEP
- removed net DIR: U$1.DIR, U$5.DIR, U$6.DIR, U$7.DIR
- removed net ESP_DSLEEP: U1.16-DSLP
- removed net FLOATS: J3.4, J4.4, J5.4, J6.4
- removed net GND: C1.-, C10.2, C12.2, C3.2, C4.-, C5.-, C6.2, C7.-, J1.GND, J3.6, J4.6, J5.6, J6.6, OKI.GND, U$1.GND@0, U$1.GND@1, U$4.GND, U$5.GND@0, U$5.GND@1, U$6.GND@0, U$6.GND@1, U$7.GND@0, U$7.GND@1, X3.GND, Y1.2
- removed net N$13: R1.2, U$4.TX
- removed net N$2: U$4.XO, Y1.3
- removed net N$29: Q1.B, R8.1
- removed net N$30: R9.1, T2.B
- removed net N$31: Q1.E, R9.2, U$4.DTR
- removed net N$4: U$4.D+, X3.D+
- removed net N$5: R8.2, T2.E, U$4.RTS
- removed net N$6: U$4.XI, Y1.1
- removed net N$7: R4.2, U$4.RX
- removed net PROBE_SCL: U1.SCL-5
- removed net PROBE_SDA: U1.SDA-4
- removed net VBUS1: D1.A, X3.VBUS
- new net 12_FLOATS: J3.4, J4.4, J5.4, J6.4, U1.12-MISO
- new net 14_A-STEP: U$6.STEP, U1.14-SCK
- new net 15_DIR: R3.2, U$1.DIR, U$5.DIR, U$6.DIR, U$7.DIR, U1.SS-15
- new net 16_B-STEP: U$1.STEP, U1.16-DSLP
- new net 4_C-STEP: U$5.STEP, U1.SDA-4
- new net 5V: D1.A, J1.1
- new net 5_D-STEP: U$7.STEP, U1.SCL-5
- net +12V: now also D2.C
- net ESP_3.3V: now also C12.1, OKI.OUT, U$1.VDD, U$5.VDD, U$6.VDD, U$7.VDD
- net ESP_FLASH: now also FLASH.1, J1.2; no longer Q1.C
- net ESP_GND: now also C1.-, C10.2, C12.2, C4.-, C5.-, C7.-, FLASH.4, J1.6, J1.7, J3.6, J4.6, J5.6, J6.6, OKI.GND, U$1.GND@0, U$1.GND@1, U$5.GND@0, U$5.GND@1, U$6.GND@0, U$6.GND@1, U$7.GND@0, U$7.GND@1, X5.2
- net ESP_RST: now also J1.3; no longer T2.C
- net ESP_RX: now also J1.4; no longer R4.1
- net ESP_TX: now also J1.5; no longer R1.1
- net N$3: now also D2.A, D4.A, X5.1; no longer U$4.D-, X3.D-
- net VCC: now also D4.C; no longer J1.PWR, U$1.VDD, U$5.VDD, U$6.VDD, U$7.VDD
Other:
- note removed: "Serial"
- moved on the sheet: D1
