File: PCB/LightManager/LightManager.brd (EAGLE design)
At the start: 100.1 x 53.1 mm, 47 parts, among them J2 RJ11, J3 RJ11, Q1 S8050, T2 S8050, U2 RT9013, X3 miniUSB, Y1 12MHz

Commit message: added panel and start of Lighting controller
Parts:
- removed C3: 10uF, microbuilder:0805-NO
- removed C6: 1uF, microbuilder:0805-NO
- removed LED1, LED2: (no value), led:SML0805
- removed R20, R21: 1k, SparkFun-Resistors:0805
- removed T2: S8050, transistor:SOT23-BEC
- removed U$4: CH340G, ch340g:SOIC16
- removed X3: miniUSB, microbuilder:USB-MINIB_LARGER
- removed Y1: 12MHz, SparkFun:RESONATOR-SMD
- added D2: 1n4148, SparkFun-DiscreteSemi:SOD-323
- added J1, J4: RJ11, SparkFun-Connectors:RJ11-6
- added J7: RJ45, SparkFun-Connectors:RJ45-8
- added Q2: IRLML2502TRPBF, freetronics-master-v1.1:SOT23-3
- added R12: 10k, LowPowerLab:0805
- added SJ1, SJ3: (no value), jumper:SJ_2
- D1: value (none) -> 1n4148
- Q1: value S8050 -> IRLML2502TRPBF; device transistor:SOT23-BEC -> freetronics-master-v1.1:SOT23-3
- R1, R4: value 470 -> 10k
- R8, R9: value 10k -> PHOTOCELLPTH; device LowPowerLab:0805 -> SparkFun-Sensors:PHOTOCELL
- moved R4 87.1 mm to (-19.1, -19.1), turned to 0 degrees
- moved D1 63.6 mm to (-24.1, -35.6)
- moved R9 59.5 mm to (-17.8, -30.5), turned to 0 degrees
- moved R8 59.1 mm to (-17.8, -24.1), turned to 0 degrees
- moved R11 52.5 mm to (21.6, 27.9)
- moved R1 47.6 mm to (-19.1, -10.2), turned to 0 degrees
- moved Q1 42.3 mm to (-19.1, -6.35), turned to 0 degrees
- moved SSR1 36.6 mm to (54.6, 66.0)
- moved SSR 33.0 mm to (54.6, 54.6)
- moved F3 29.6 mm to (83.8, 73.7)
- moved U$1 26.8 mm to (87.6, 43.2)
- moved MAINS2 26.5 mm to (94.0, 64.8), turned to 270 degrees
- moved F1 18.2 mm to (96.5, 25.4)
- moved MAINS1 17.6 mm to (94.0, 45.7), turned to 270 degrees
- moved C5 12.8 mm to (43.2, 22.9)
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Connections:
- removed net +3V3: C3.1, C6.1, U$4.16, U$4.4
- removed net AC-L: F1.P$1, U$9.P$2
- removed net AC-N: R2.1, U$1.AC1, U$9.P$1
- removed net AIR_PUMP_BB: R21.1, SSR1.+
- removed net ESP_5V: D1.1
- removed net ESP_TX_2: R1.1
- removed net FEED_PUMP_BB: R20.1, SSR.+
- removed net GND_BB: LED1.C, LED2.C, SSR.-, SSR1.-
- removed net N$13: R1.2, U$4.2
- removed net N$29: Q1.B, R8.1
- removed net N$30: R9.1, T2.B
- removed net N$31: Q1.E, R9.2, U$4.13
- removed net N$43: LED1.A, R20.2
- removed net N$50: LED2.A, R21.2
- removed net VBUS1: D1.2, X3.VBUS
- new net ADC: J1.3, J4.3, U1.ADC
- new net ADC_EXT: D1.1, D2.1, R12.2
- new net D6_C_SSR: Q1.1, Q2.1, R1.2, R4.2
- new net FLOAT1: J2.4, SJ1.1, SJ3.1
- new net FLOAT2: J3.4, SJ1.3, SJ3.3
- new net FLOATS_EXT: R8.2
- new net LIGHT1: J1.2
- new net LIGHT2: J4.2
- new net N$11: R9.2
- new net VCC: C5.+, C8.1, J7.1, R10.1, R11.2, SSR.+, SSR1.+, U2.1
- net 12_TEMP: now also J1.5, J4.5
- net 5V: now also J1.1, J2.1, J3.1, J4.1; no longer C5.+, C8.1, R10.1, R11.2, U2.1
- net ESP_FLASH: now also J7.2; no longer Q1.C
- net ESP_RST: now also J7.3; no longer T2.C
- net ESP_RX: now also J7.4; no longer R4.1
- net ESP_TX: now also J7.5
- net GND: now also J1.6, J4.6, J7.6, J7.7, Q1.2, Q2.2, R1.1, R12.1, R4.1; no longer C3.2, C6.2, U$4.1, X3.GND, X3.GND1, X3.GND2, X3.GND3, X3.GND4, Y1.2
- net MAIN_ACTIVE: now also F1.P$1, U$9.P$2
- net MAIN_NETURAL: now also R2.1, U$1.AC1, U$9.P$1
- net N$2: now also D2.2, R8.1; no longer U$4.8, Y1.3
- net N$3: now also Q1.3, SSR.-; no longer U$4.6, X3.D-
- net N$4: now also Q2.3, SSR1.-; no longer U$4.5, X3.D+
- net N$5: now also D1.2, R9.1; no longer R8.2, T2.E, U$4.14
- net N$6: now also J1.4, SJ1.2; no longer U$4.7, Y1.1
- net N$7: now also J4.4, SJ3.2; no longer R4.2, U$4.3
Other:
- board size 100.1 x 53.1 mm -> 100.3 x 100.3 mm
