File: PCB/LightManager/LightManager.sch (EAGLE design)
At the start: 46 parts, among them J2 RJ11, J3 RJ11, Q1 S8050, T2 S8050, U2 RT9013, X3 miniUSB, Y1 12MHz

Commit message: added panel and start of Lighting controller
Parts:
- removed C3: 10uF, microbuilder:CAP_CERAMIC0805-NOOUTLINE
- removed C6: 1uF, microbuilder:CAP_CERAMIC0805-NOOUTLINE
- removed LED1, LED2: (no value), led:LEDSML0805
- removed R20, R21: 1k, SparkFun-Resistors:RESISTOR0805-RES
- removed T2: S8050, transistor:BC817-16LT1-NPN-SOT23-BEC
- removed U$4: CH340G, ch340g:CH340G
- removed X3: miniUSB, microbuilder:USBMINIBLARGE
- removed Y1: 12MHz, SparkFun:RESONATORSMD
- added D2: 1n4148, SparkFun-DiscreteSemi:DIODESOD
- added J1, J4: RJ11, SparkFun-Connectors:RJ11-6
- added J7: RJ45, SparkFun-Connectors:RJ45-8
- added Q2: IRLML2502TRPBF, freetronics-master-v1.1:MOSFET-NCHANNELSMD
- added R12: 10k, LowPowerLab:RESISTOR0805
- added SJ1, SJ3: (no value), jumper:SJ2W
- D1: value (none) -> 1n4148
- Q1: value S8050 -> IRLML2502TRPBF; device transistor:BC817-16LT1-NPN-SOT23-BEC -> freetronics-master-v1.1:MOSFET-NCHANNELSMD
- R1, R4: value 470 -> 10k
- R8, R9: value 10k -> PHOTOCELLPTH; device LowPowerLab:RESISTOR0805 -> SparkFun-Sensors:PHOTOCELLPTH
Connections:
- removed net +3V3: C3.1, C6.1, U$4.V3, U$4.VCC
- removed net AC-L: F1.1, U$9.P$2
- removed net AC-N: R2.1, U$1.AC1, U$9.P$1
- removed net AIR_PUMP_BB: R21.1, SSR1.A
- removed net ESP_5V: D1.C
- removed net ESP_TX_2: R1.1
- removed net FEED_PUMP_BB: R20.1, SSR.A
- removed net GND_BB: LED1.C, LED2.C, SSR.K, SSR1.K
- removed net N$13: R1.2, U$4.TX
- removed net N$29: Q1.B, R8.1
- removed net N$30: R9.1, T2.B
- removed net N$31: Q1.E, R9.2, U$4.DTR
- removed net N$43: LED1.A, R20.2
- removed net N$50: LED2.A, R21.2
- removed net VBUS1: D1.A, X3.VBUS
- new net ADC: J1.3, J4.3, U1.ADC
- new net ADC_EXT: D1.C, D2.C, R12.2
- new net D6_C_SSR: Q1.G, Q2.G, R1.2, R4.2
- new net FLOAT1: J2.4, SJ1.1, SJ3.1
- new net FLOAT2: J3.4, SJ1.3, SJ3.3
- new net FLOATS_EXT: R8.P$2
- new net LIGHT1: J1.2
- new net LIGHT2: J4.2
- new net N$11: R9.P$2
- new net VCC: C5.+, C8.1, J7.1, R10.1, R11.2, SSR.A, SSR1.A, U2.IN
- net 12_TEMP: now also J1.5, J4.5
- net 5V: now also J1.1, J2.1, J3.1, J4.1; no longer C5.+, C8.1, R10.1, R11.2, U2.IN
- net ESP_FLASH: now also J7.2; no longer Q1.C
- net ESP_RST: now also J7.3; no longer T2.C
- net ESP_RX: now also J7.4; no longer R4.1
- net ESP_TX: now also J7.5
- net GND: now also J1.6, J4.6, J7.6, J7.7, Q1.S, Q2.S, R1.1, R12.1, R4.1; no longer C3.2, C6.2, U$4.GND, X3.GND, Y1.2
- net MAIN_ACTIVE: now also F1.1, U$9.P$2
- net MAIN_NETURAL: now also R2.1, U$1.AC1, U$9.P$1
- net N$2: now also D2.A, R8.P$1; no longer U$4.XO, Y1.3
- net N$3: now also Q1.D, SSR.K; no longer U$4.D-, X3.D-
- net N$4: now also Q2.D, SSR1.K; no longer U$4.D+, X3.D+
- net N$5: now also D1.A, R9.P$1; no longer R8.2, T2.E, U$4.RTS
- net N$6: now also J1.4, SJ1.2; no longer U$4.XI, Y1.1
- net N$7: now also J4.4, SJ3.2; no longer R4.2, U$4.RX
Other:
- note added: "1 = 5v 2 = 3v3 3 = ??? 4 = Floats 5 = Temps 6 = GND"
- note added: "Flow Sensor: pin 1 for pwr Pin 2 for Sensor (2 x GPIO) Float Sensor: pin 4 (2 x GPIO) Temps & Lights: Pin 5 for Temp (1 x GPIO) Pin 2 for pwr (2 x GPIO) Pin 3 for reading (ADC)"
- note added: "Light/Flow/Pings"
- note added: "Temp/Float"
- note removed: "Temp"
- moved on the sheet: C5, D1, F1, R1, R10, R16, R2, R4
