File: PCB/SensorManager/SensorManager.brd (EAGLE design)
At the start: 100.1 x 41.7 mm, 52 parts, among them J1 POWER_JACKPTH_LOCK, J2 RJ11, Q1 S8050, T2 S8050, U2 RT9013, X3 miniUSB, Y1 12MHz

Commit message: added panel and start of Lighting controller
Parts:
- removed C36, C9: 0.1uF, SparkFun-Capacitors:0805
- removed C4, C5: 1uF, SparkFun-Capacitors:0805
- removed D1, D2: (no value), SparkFun-DiscreteSemi:SOD-323
- removed J1: POWER_JACKPTH_LOCK, SparkFun-Connectors:POWER_JACK_PTH_LOCK
- removed L2: WS2812B, adafruit:WS2812B
- removed Q1, T2: S8050, transistor:SOT23-BEC
- removed R13, R3, R5, R6, R7: 10k, LowPowerLab:0805
- removed R43: 100, LowPowerLab:0805
- removed U$10, U$7: SI860X, 1_Skips:SO08
- removed U$2: BNCPTH, SparkFun-Connectors:BNC
- removed U$20: (no value), 11_Skips_Refactor:ID_LOGO_X0.25
- removed U$6: R1SE-3.33.3, 1_Skips:R1SE-0505
- removed U1: (no value), esp8266modules:ESP12-SMD
- removed X3: miniUSB, microbuilder:USB-MINIB_LARGER
- removed Y1: 12MHz, SparkFun:RESONATOR-SMD
- added C11: 1uF, SparkFun-Capacitors:0805
- added C13: 0.1uF, SparkFun-Capacitors:0805
- added C14: 10uF, adafruit:153CLV-0405
- added D3: (no value), SparkFun-DiscreteSemi:SOD-323
- added D5: B120B-13-F, SparkFun-DiscreteSemi:SMB-DIODE
- added FLASH1: (no value), SparkFun-Electromechanical:TACTILE_SWITCH_SMD
- added J7: RJ45, SparkFun-Connectors:RJ45-8
- added J8: (no value), SparkFun-Connectors:1X02
- added J9: RJ11, SparkFun-Connectors:RJ11-6
- added L1: WS2812B, adafruit:WS2812B
- added OLED: (no value), SparkFun-Connectors:1X04
- added Q3: IRLML2502TRPBF, freetronics-master-v1.1:SOT23-3
- added R17: 33, LowPowerLab:0805
- added R18, R19: 4k7, LowPowerLab:0805
- added R2, R22: 10k, LowPowerLab:0805
- added S1: ENCODER-SWITCH, SparkFun-Switches:ROTARY_ENC_PLAIN
- added U$11: SI860X, 1_Skips:SO08
- added U$12: LOGO_GROBOTICS, 1_Skips:GROBOTICS
- added U$13: (no value), 11_Skips_Refactor:ID_LOGO_X0.25
- added U$14: MURATA-DCDC, 11_Skips_Refactor:MURATA_DCDC
- added U$3: BNCPTH, SparkFun-Connectors:BNC
- added U3: RT9013, SparkFun-IC-Power:SOT23-5
- added X1: (no value), con-conrad:733980-62
- C3: value 10uF -> 1uF; device microbuilder:0805-NO -> SparkFun-Capacitors:0805
- C6: value 1uF -> 0.1uF; device microbuilder:0805-NO -> SparkFun-Capacitors:0805
- R1, R4: value 470 -> 10k
- R9: value 10k -> 100
- U$4: value CH340G -> MURATA-DCDC; device ch340g:SOIC16 -> 11_Skips_Refactor:MURATA_DCDC
- U$8: value BNCPTH -> SI860X; device SparkFun-Connectors:BNC -> 1_Skips:SO08
- U$9: value R1SE-3.33.3 -> BNCPTH; device 1_Skips:R1SE-0505 -> SparkFun-Connectors:BNC
- U2: value RT9013 -> (none); device SparkFun-IC-Power:SOT23-5 -> esp8266modules:ESP12-SMD
- moved U$4 58.5 mm to (87.6, 19.1)
- moved C3 55.5 mm to (69.8, 30.5), turned to 0 degrees
- moved U$8 44.7 mm to (87.6, 35.5), turned to 90 degrees
- moved J2 42.0 mm to (44.5, 5.08)
- moved R16 40.7 mm to (45.7, 16.5), turned to 180 degrees
- moved C2 39.4 mm to (50.5, 28.3), turned to 90 degrees
- moved U2 36.2 mm to (37.5, 36.2), flipped to the bottom, turned to 0 degrees
- moved R9 26.9 mm to (40.6, 28.1), turned to 0 degrees
- moved C8 26.6 mm to (31.3, 24.6), turned to 270 degrees
- moved R1 24.0 mm to (47.6, 33.5)
- moved C16 23.2 mm to (34.3, 24.1), turned to 270 degrees
- moved C6 17.4 mm to (35.2, 33.7), turned to 180 degrees
- moved R4 17.3 mm to (34.0, 30.8), turned to 0 degrees
- moved R8 15.8 mm to (34.1, 28.9), turned to 0 degrees
- moved U$9 14.8 mm to (63.5, 10.2), turned to 180 degrees
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Connections:
- removed net +3V3: C3.1, C6.1, U$4.16, U$4.4
- removed net 13_WS2812: R43.2, U1.GPIO13
- removed net 15: R3.2, U1.GPIO15
- removed net 5V: C8.1, D1.1, D2.1, R12.1, U2.1
- removed net B0_ENC_BTN: R13.1, U1.GPIO2
- removed net ESP_3.3V: C16.1, C2.1, C36.2, C9.2, L2.1-VDD, R13.2, R5.2, R6.2, R7.2, U1.VCC, U2.5
- removed net ESP_DSLEEP: U1.GPIO16
- removed net ESP_FLASH: Q1.C, R7.1, U1.GPIO0
- removed net ESP_GND: C36.1, C9.1, L2.3-GND, R3.1, U1.GND
- removed net ESP_RST: R5.1, T2.C, U1.RESET
- removed net ESP_RX: R4.1, U1.TXD0
- removed net ESP_TX: R1.1, U1.RXD0
- removed net N$1: R6.1, U1.CH_PD
- removed net N$18: EC1.PRB, U$8.S
- removed net N$22: EC1.PRA, U$8.GND
- removed net N$23: EC1.RX, R15.1, U$10.6
- removed net N$24: EC1.TX, R14.1, U$10.7
- removed net N$3: U$4.6, X3.D-
- removed net N$30: R9.1, T2.B
- removed net N$31: Q1.E, R9.2, U$4.13
- removed net N$74: L2.4-DIN, R43.1
- removed net N$9: EC.PRB, U$2.S
- removed net VBUS1: D1.2, X3.VBUS
- new net 13_WS2812_SENSOR: R9.2, U2.GPIO13
- new net 15_FF: R17.1, U2.GPIO15
- new net 16_DSLEEP: S1.B, U2.GPIO16
- new net 2: R8.1, U2.GPIO2
- new net 5V_SENSOR: C11.1, D3.1, J7.1, R12.1, U3.1
- new net ESP_FLASH_SENSOR: FLASH1.1, J7.2, R4.1, S1.SW+, U2.GPIO0
- new net ESP_RST_SENSOR: J7.3, R1.1, U2.RESET
- new net ESP_RX_SENSOR: J7.4, U2.TXD0
- new net ESP_TX_SENSOR: J7.5, U2.RXD0
- new net N$19: Q3.1, R17.2, R22.2
- new net VCC_SENSOR: C14.+, D3.2, D5.C, J8.1, X1.1
- net 12_TEMP: now also J9.5, U2.GPIO12; no longer U1.GPIO12
- net 14_SCK: now also S1.A, U2.GPIO14; no longer U1.GPIO14
- net 3.3V: now also C13.2, C16.1, C2.1, C3.1, C6.2, C8.1, J9.2, L1.1-VDD, OLED.1, R1.2, R18.2, R19.2, R2.2, R4.2, R8.2, U$11.1, U$14.VIN+, U$4.VIN+, U$8.1, U2.VCC, U3.5; no longer C4.1, C5.1, U$10.1, U$6.VCC, U$7.1, U$9.VCC
- net GND: now also C11.2, C13.1, C14.-, C6.1, FLASH1.4, J7.6, J7.7, J9.6, L1.3-GND, OLED.2, Q3.2, R22.1, S1.C, S1.SW-, U$11.4, U$14.VIN-, U$4.VIN-, U$8.4, U2.GND, U3.2, X1.2; no longer C4.2, C5.2, C6.2, J1.GND, U$10.4, U$4.1, U$6.GND, U$7.4, U$9.GND, U2.2, X3.GND, X3.GND1, X3.GND2, X3.GND3, X3.GND4, Y1.2
- net N$10: now also R2.1, U2.CH_PD; no longer R12.2, U2.3
- net N$11: now also L1.4-DIN, R9.1; no longer D2.2, J1.PWR
- net N$12: now also U$8.6; no longer U$7.6
- net N$13: now also R12.2, U3.3; no longer R1.2, U$4.2
- net N$14: now also U$8.7; no longer U$7.7
- net N$15: now also U$4.VOUT-, U$8.5; no longer U$6.ISO_GND, U$7.5
- net N$16: now also U$4.VOUT+, U$8.8; no longer U$6.ISO_VCC, U$7.8
- net N$17: now also U$11.5, U$14.VOUT-; no longer U$10.5, U$9.ISO_GND
- net N$2: now also EC.PRB, U$3.S; no longer U$4.8, Y1.3
- net N$25: now also U$11.8, U$14.VOUT+; no longer U$10.8, U$9.ISO_VCC
- net N$29: now also D5.A, J8.2, Q3.3; no longer Q1.B, R8.1
- net N$4: now also EC1.PRB, U$9.S; no longer U$4.5, X3.D+
- net N$5: now also EC1.PRA, U$9.GND; no longer R8.2, T2.E, U$4.14
- net N$6: now also EC1.RX, R15.1, U$11.6; no longer U$4.7, Y1.1
- net N$7: now also EC1.TX, R14.1, U$11.7; no longer R4.2, U$4.3
- net N$8: now also U$3.GND; no longer U$2.GND
- net PROBE_SCL: now also OLED.3, R18.1, U$11.3, U$8.3, U2.GPIO5; no longer U$10.3, U$7.3, U1.GPIO5
- net PROBE_SDA: now also OLED.4, R19.1, U$11.2, U$8.2, U2.GPIO4; no longer U$10.2, U$7.2, U1.GPIO4
Routing:
- net 3.3V: track 90.3 -> 221.7 mm
- net VCC_SENSOR: track 0.00 -> 121.3 mm
- net 15_FF: track 0.00 -> 94.0 mm, vias 0 -> 1
- net ESP_RST_SENSOR: track 0.00 -> 69.2 mm, vias 0 -> 2
- net PROBE_SDA: track 51.8 -> 111.5 mm, vias 3 -> 4
- net ESP_FLASH_SENSOR: track 0.00 -> 40.3 mm, vias 0 -> 2
- net PROBE_SCL: track 48.8 -> 88.3 mm, vias 3 -> 4
- net 12_TEMP: track 0.00 -> 39.2 mm
- net ESP_TX_SENSOR: track 0.00 -> 38.0 mm
- net ESP_RX_SENSOR: track 0.00 -> 29.4 mm, vias 0 -> 2
- net GND: track 122.5 -> 149.7 mm, vias 5 -> 13
- net 14_SCK: track 0.00 -> 22.1 mm, vias 0 -> 1
- net N$16: track 19.6 -> 41.4 mm
- net 16_DSLEEP: track 0.00 -> 21.8 mm, vias 0 -> 1
- net N$25: track 19.6 -> 40.1 mm
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- added copper zone on layer 1, net GND
- added copper zone on layer 16, net GND
Other:
- board size 100.1 x 41.7 mm -> 100.3 x 43.2 mm
- board text added: "6/24/17"
- board text added: "FLASH"
- board text added: "Rx"
- board text added: "Tx"
- board text added: "Water Quality v1 Grobotics.io"
