File: PCB/SensorManager/SensorManager.sch (EAGLE design)
At the start: 51 parts, among them J1 POWER_JACKPTH_LOCK, J2 RJ11, Q1 S8050, T2 S8050, U2 RT9013, X3 miniUSB, Y1 12MHz

Commit message: added panel and start of Lighting controller
Parts:
- removed C4, C5: 1uF, SparkFun-Capacitors:CAP0805
- removed C9: 0.1uF, SparkFun-Capacitors:CAP0805
- removed D1, D2: (no value), SparkFun-DiscreteSemi:DIODESOD
- removed J1: POWER_JACKPTH_LOCK, SparkFun-Connectors:POWER_JACKPTH_LOCK
- removed Q1, T2: S8050, transistor:BC817-16LT1-NPN-SOT23-BEC
- removed R13, R3, R5, R7: 10k, LowPowerLab:RESISTOR0805
- removed R43: 100, LowPowerLab:RESISTOR0805
- removed U$6: R1SE-3.33.3, 1_Skips:R1SE-0505
- removed U$7: SI860X, 1_Skips:SI860X
- removed U1: (no value), esp8266modules:ESP12SMD
- removed X3: miniUSB, microbuilder:USBMINIBLARGE
- removed Y1: 12MHz, SparkFun:RESONATORSMD
- added C11: 1uF, SparkFun-Capacitors:CAP0805
- added C14: 10uF, adafruit:CPOL-US153CLV-0405
- added D3: (no value), SparkFun-DiscreteSemi:DIODESOD
- added D5: B120B-13-F, SparkFun-DiscreteSemi:DIODESMB
- added FLASH1: (no value), SparkFun-Electromechanical:TAC_SWITCHSMD
- added J7: RJ45, SparkFun-Connectors:RJ45-8
- added J8: (no value), SparkFun-Connectors:CONN_02
- added J9: RJ11, SparkFun-Connectors:RJ11-6
- added OLED: (no value), SparkFun-Connectors:CONN_04
- added Q3: IRLML2502TRPBF, freetronics-master-v1.1:MOSFET-NCHANNELSMD
- added R17: 33, LowPowerLab:RESISTOR0805
- added R18, R19: 4k7, LowPowerLab:RESISTOR0805
- added R22: 10k, LowPowerLab:RESISTOR0805
- added S1: ENCODER-SWITCH, SparkFun-Switches:ENCODER-SWITCH
- added U$12: LOGO_GROBOTICS, 1_Skips:LOGO_GROBOTICS
- added U$14: MURATA-DCDC, 11_Skips_Refactor:MURATA-DCDC
- added U3: RT9013, SparkFun-IC-Power:AP2202-ADJ
- added X1: (no value), con-conrad:733980-62
- C3: value 10uF -> 1uF; device microbuilder:CAP_CERAMIC0805-NOOUTLINE -> SparkFun-Capacitors:CAP0805
- C6: value 1uF -> 0.1uF; device microbuilder:CAP_CERAMIC0805-NOOUTLINE -> SparkFun-Capacitors:CAP0805
- R1, R4: value 470 -> 10k
- R9: value 10k -> 100
- U$4: value CH340G -> MURATA-DCDC; device ch340g:CH340G -> 11_Skips_Refactor:MURATA-DCDC
- U$8: value BNCPTH -> SI860X; device SparkFun-Connectors:BNCPTH -> 1_Skips:SI860X
- U$9: value R1SE-3.33.3 -> BNCPTH; device 1_Skips:R1SE-0505 -> SparkFun-Connectors:BNCPTH
- U2: value RT9013 -> (none); device SparkFun-IC-Power:AP2202-ADJ -> esp8266modules:ESP12SMD
- renumbered C36 to C13, L2 to L1, R6 to R2, U$10 to U$11, U$2 to U$3
Connections:
- removed net +3V3: C3.1, C6.1, U$4.V3, U$4.VCC
- removed net 13_WS2812: R43.2, U1.13-MOSI
- removed net 15: R3.2, U1.SS-15
- removed net 5V: C8.1, D1.C, D2.C, R12.1, U2.IN
- removed net B0_ENC_BTN: R13.1, U1.2
- removed net ESP_3.3V: C13.2, C16.1, C2.1, C9.2, L1.VDD, R13.2, R2.2, R5.2, R7.2, U1.VCC, U2.OUT
- removed net ESP_DSLEEP: U1.16-DSLP
- removed net ESP_FLASH: Q1.C, R7.1, U1.FLASH-0
- removed net ESP_GND: C13.1, C9.1, L1.GND, R3.1, U1.GND
- removed net ESP_RST: R5.1, T2.C, U1.RESET
- removed net ESP_RX: R4.1, U1.TX-1
- removed net ESP_TX: R1.1, U1.RX-3
- removed net N$1: R2.1, U1.CH_PD
- removed net N$18: EC1.PRB, U$8.OUT
- removed net N$2 (its old number): U$4.XO, Y1.3
- removed net N$22: EC1.PRA, U$8.GND
- removed net N$3: U$4.D-, X3.D-
- removed net N$30: R9.1, T2.B
- removed net N$31: Q1.E, R9.2, U$4.DTR
- removed net N$6 (its old number): U$4.XI, Y1.1
- removed net N$7 (its old number): R4.2, U$4.RX
- removed net N$74: L1.DIN, R43.1
- removed net VBUS1: D1.A, X3.VBUS
- new net 13_WS2812_SENSOR: R9.2, U2.13-MOSI
- new net 15_FF: R17.1, U2.SS-15
- new net 16_DSLEEP: S1.B, U2.16-DSLP
- new net 2: R8.1, U2.2
- new net 5V_SENSOR: C11.1, D3.C, J7.1, R12.1, U3.IN
- new net ESP_FLASH_SENSOR: FLASH1.1, J7.2, R4.1, S1.SW+, U2.FLASH-0
- new net ESP_RST_SENSOR: J7.3, R1.1, U2.RESET
- new net ESP_RX_SENSOR: J7.4, U2.TX-1
- new net ESP_TX_SENSOR: J7.5, U2.RX-3
- new net N$19: Q3.G, R17.2, R22.2
- new net VCC_SENSOR: C14.+, D3.A, D5.C, J8.1, X1.1
- net 12_TEMP: now also J9.5, U2.12-MISO; no longer U1.12-MISO
- net 14_SCK: now also S1.A, U2.14-SCK; no longer U1.14-SCK
- net 3.3V: now also C13.2, C16.1, C2.1, C3.1, C6.2, C8.1, J9.2, L1.VDD, OLED.1, R1.2, R18.2, R19.2, R2.2, R4.2, R8.2, U$14.VIN+, U$4.VIN+, U$8.VCC, U2.VCC, U3.OUT; no longer C4.1, C5.1, U$6.VCC, U$7.VCC, U$9.VCC
- net GND: now also C11.2, C13.1, C14.-, C6.1, FLASH1.4, J7.6, J7.7, J9.6, L1.GND, OLED.2, Q3.S, R22.1, S1.C, S1.SW-, U$14.VIN-, U$4.VIN-, U$8.GND, U3.GND, X1.2; no longer C4.2, C5.2, C6.2, J1.GND, U$4.GND, U$6.GND, U$7.GND, U$9.GND, X3.GND, Y1.2
- net N$10: now also R2.1, U2.CH_PD; no longer R12.2, U2.EN
- net N$11: now also L1.DIN, R9.1; no longer D2.A, J1.PWR
- net N$12: now also U$8.ISO_SCL; no longer U$7.ISO_SCL
- net N$13: now also R12.2, U3.EN; no longer R1.2, U$4.TX
- net N$14: now also U$8.ISO_SDA; no longer U$7.ISO_SDA
- net N$15: now also U$4.VOUT-, U$8.ISO_GND; no longer U$6.ISO_GND, U$7.ISO_GND
- net N$16: now also U$4.OUT+, U$8.ISO_VCC; no longer U$6.ISO_VCC, U$7.ISO_VCC
- net N$17: now also U$14.VOUT-; no longer U$9.ISO_GND
- net N$25: now also U$14.OUT+; no longer U$9.ISO_VCC
- net N$29: now also D5.A, J8.2, Q3.D; no longer Q1.B, R8.1
- net N$4: now also EC1.PRB, U$9.OUT; no longer U$4.D+, X3.D+
- net N$5: now also EC1.PRA, U$9.GND; no longer R8.2, T2.E, U$4.RTS
- net PROBE_SCL: now also OLED.3, R18.1, U$8.SCL, U2.SCL-5; no longer U$7.SCL, U1.SCL-5
- net PROBE_SDA: now also OLED.4, R19.1, U$8.SDA, U2.SDA-4; no longer U$7.SDA, U1.SDA-4
Other:
- note added: "15 should be pulled low We do it at the MOSFET"
- moved on the sheet: C2, C3, C6, C8, R1, R4, R8, R9
